Commit message: asdfghj

File: src/mobile_base_description/urdf/gazebo.xacro (robot description, xacro)
@@ -1,22 +1,22 @@
-<gazebo>
-  <plugin name='diff_drive' filename='libgazebo_ros_diff_drive.so'>
-    <ros>
-      <namespace>/demo</namespace>
-    </ros>
-    <!-- wheels -->
-    <left_joint>left_wheel_joint</left_joint>
-    <right_joint>right_wheel_joint</right_joint>
-    <!-- kinematics -->
-    <wheel_separation>0.269</wheel_separation>
-    <wheel_diameter>0.26</wheel_diameter>
-    <!-- limits -->
-    <max_wheel_torque>20</max_wheel_torque>
-    <max_wheel_acceleration>1.0</max_wheel_acceleration>
-    <!-- output -->
-    <publish_odom>true</publish_odom>
-    <publish_odom_tf>false</publish_odom_tf>
-    <publish_wheel_tf>true</publish_wheel_tf>
-    <odometry_frame>odom</odometry_frame>
-    <robot_base_frame>base_link</robot_base_frame>
-  </plugin>
-</gazebo>
+<?xml version="1.0"?>
+<robot xmlns:xacro="http://www.ros.org/wiki/xacro">
+  <gazebo>
+    <plugin name='diff_drive' filename='libgazebo_ros_diff_drive.so'>
+      <!-- wheels -->
+      <left_joint>left_wheel_joint</left_joint>
+      <right_joint>right_wheel_joint</right_joint>
+      <!-- kinematics -->
+      <wheel_separation>0.269</wheel_separation>
+      <wheel_diameter>0.26</wheel_diameter>
+      <!-- limits -->
+      <max_wheel_torque>20</max_wheel_torque>
+      <max_wheel_acceleration>1.0</max_wheel_acceleration>
+      <!-- output -->
+      <publish_odom>true</publish_odom>
+      <publish_odom_tf>true</publish_odom_tf>
+      <publish_wheel_tf>true</publish_wheel_tf>
+      <odometry_frame>odom</odometry_frame>
+      <robot_base_frame>base_link</robot_base_frame>
+    </plugin>
+  </gazebo>
+</robot>

File: src/mobile_base_description/urdf/mobile_base.urdf.xacro (robot description, xacro)
@@ -27,5 +27,5 @@
       <geometry>
         <mesh
-          filename="package://mobile_base_description/meshes/base_link.STL" />
+          filename="file://$(find mobile_base_description)/meshes/base_link.STL" />
       </geometry>
       <material
@@ -41,5 +41,5 @@
       <geometry>
         <mesh
-          filename="package://mobile_base_description/meshes/base_link.STL" />
+          filename="file://$(find mobile_base_description)/meshes/base_link.STL" />
       </geometry>
     </collision>
@@ -67,19 +67,19 @@
       <geometry>
         <mesh
-          filename="package://mobile_base_description/meshes/left_wheel.STL" />
-      </geometry>
-      <material
-        name="">
-        <color
-          rgba="0.792156862745098 0.819607843137255 0.933333333333333 1" />
-      </material>
-    </visual>
-    <collision>
-      <origin
-        xyz="0 0 0"
-        rpy="0 0 0" />
-      <geometry>
-        <mesh
-          filename="package://mobile_base_description/meshes/left_wheel.STL" />
+          filename="file://$(find mobile_base_description)/meshes/left_wheel.STL" />
+      </geometry>
+      <material
+        name="">
+        <color
+          rgba="0.792156862745098 0.819607843137255 0.933333333333333 1" />
+      </material>
+    </visual>
+    <collision>
+      <origin
+        xyz="0 0 0"
+        rpy="0 0 0" />
+      <geometry>
+        <mesh
+          filename="file://$(find mobile_base_description)/meshes/left_wheel.STL" />
       </geometry>
     </collision>
@@ -120,19 +120,19 @@
       <geometry>
         <mesh
-          filename="package://mobile_base_description/meshes/right_wheel.STL" />
-      </geometry>
-      <material
-        name="">
-        <color
-          rgba="0.792156862745098 0.819607843137255 0.933333333333333 1" />
-      </material>
-    </visual>
-    <collision>
-      <origin
-        xyz="0 0 0"
-        rpy="0 0 0" />
-      <geometry>
-        <mesh
-          filename="package://mobile_base_description/meshes/right_wheel.STL" />
+          filename="file://$(find mobile_base_description)/meshes/right_wheel.STL" />
+      </geometry>
+      <material
+        name="">
+        <color
+          rgba="0.792156862745098 0.819607843137255 0.933333333333333 1" />
+      </material>
+    </visual>
+    <collision>
+      <origin
+        xyz="0 0 0"
+        rpy="0 0 0" />
+      <geometry>
+        <mesh
+          filename="file://$(find mobile_base_description)/meshes/right_wheel.STL" />
       </geometry>
     </collision>
@@ -173,19 +173,19 @@
       <geometry>
         <mesh
-          filename="package://mobile_base_description/meshes/camera.STL" />
-      </geometry>
-      <material
-        name="">
-        <color
-          rgba="0.792156862745098 0.819607843137255 0.933333333333333 1" />
-      </material>
-    </visual>
-    <collision>
-      <origin
-        xyz="0 0 0"
-        rpy="0 0 0" />
-      <geometry>
-        <mesh
-          filename="package://mobile_base_description/meshes/camera.STL" />
+          filename="file://$(find mobile_base_description)/meshes/camera.STL" />
+      </geometry>
+      <material
+        name="">
+        <color
+          rgba="0.792156862745098 0.819607843137255 0.933333333333333 1" />
+      </material>
+    </visual>
+    <collision>
+      <origin
+        xyz="0 0 0"
+        rpy="0 0 0" />
+      <geometry>
+        <mesh
+          filename="file://$(find mobile_base_description)/meshes/camera.STL" />
       </geometry>
     </collision>
@@ -226,19 +226,19 @@
       <geometry>
         <mesh
-          filename="package://mobile_base_description/meshes/laser.STL" />
-      </geometry>
-      <material
-        name="">
-        <color
-          rgba="0.792156862745098 0.819607843137255 0.933333333333333 1" />
-      </material>
-    </visual>
-    <collision>
-      <origin
-        xyz="0 0 0"
-        rpy="0 0 0" />
-      <geometry>
-        <mesh
-          filename="package://mobile_base_description/meshes/laser.STL" />
+          filename="file://$(find mobile_base_description)/meshes/laser.STL" />
+      </geometry>
+      <material
+        name="">
+        <color
+          rgba="0.792156862745098 0.819607843137255 0.933333333333333 1" />
+      </material>
+    </visual>
+    <collision>
+      <origin
+        xyz="0 0 0"
+        rpy="0 0 0" />
+      <geometry>
+        <mesh
+          filename="file://$(find mobile_base_description)/meshes/laser.STL" />
       </geometry>
     </collision>

File: src/mobile_base_description/urdf/mobile_base_gazebo.xacro (robot description, xacro)
@@ -1,9 +1,9 @@
 <?xml version="1.0"?>
 <robot xmlns:xacro="http://www.ros.org/wiki/xacro" name="mobile_base">
-    <xacro:arg name="initial_positions_file" default="initial_positions.yaml" />
     <!-- Import panda urdf file -->
     <xacro:include filename="$(find mobile_base_description)/urdf/mobile_base.urdf.xacro" />
      <!-- Import panda urdf file -->
     <xacro:include filename="$(find mobile_base_description)/urdf/base_footprint.xacro" />
+    <xacro:include filename="$(find mobile_base_description)/urdf/ros2_control.xacro" />
     <xacro:include filename="$(find mobile_base_description)/urdf/gazebo.xacro" />
 </robot>

Commit message: sd

File: src/mobile_base_description/urdf/gazebo.xacro (robot description, xacro)
@@ -3,4 +3,5 @@
   <gazebo>
     <plugin name='diff_drive' filename='libgazebo_ros_diff_drive.so'>
+      <!--namspce can be used-->
       <!-- wheels -->
       <left_joint>left_wheel_joint</left_joint>
@@ -20,3 +21,7 @@
     </plugin>
   </gazebo>
+  <gazebo reference="base_link">
+        <mu1 value="0.001"/>
+        <mu2 value="0.001"/>
+  </gazebo>
 </robot>

File: src/mobile_base_description/urdf/lidar.xacro (robot description, xacro)
@@ -1,33 +1,5 @@
 <?xml version="1.0"?>
 <robot xmlns:xacro="http://www.ros.org/wiki/xacro" >
-    <joint name="laser_joint" type="fixed">
-        <parent link="chassis"/>
-        <child link="laser_frame"/>
-        <origin xyz="0.122 0 0.212" rpy="0 0 0"/>
-    </joint>
-    <link name="laser_frame">
-        <visual>
-            <geometry>
-                <cylinder radius="0.05" length="0.04"/>
-            </geometry>
-            <material name="black"/>
-        </visual>
-        <visual>
-            <origin xyz="0 0 -0.05"/>
-            <geometry>
-                <cylinder radius="0.01" length="0.1"/>
-            </geometry>
-            <material name="black"/>
-        </visual>
-        <collision>
-            <geometry>
-                <cylinder radius="0.05" length="0.04"/>
-            </geometry>
-        </collision>
-        <xacro:inertial_cylinder mass="0.1" length="0.04" radius="0.05">
-            <origin xyz="0 0 0" rpy="0 0 0"/>
-        </xacro:inertial_cylinder>
-    </link>
-    <gazebo reference="laser_frame">
+    <gazebo reference="laser">
         <material>Gazebo/Black</material>
         <sensor name="laser" type="ray">
@@ -53,5 +25,5 @@
                 </ros>
                 <output_type>sensor_msgs/LaserScan</output_type>
-                <frame_name>laser_frame</frame_name>
+                <frame_name>laser</frame_name>
             </plugin>
         </sensor>

File: src/mobile_base_description/urdf/mobile_base_gazebo.xacro (robot description, xacro)
@@ -7,3 +7,4 @@
     <xacro:include filename="$(find mobile_base_description)/urdf/ros2_control.xacro" />
     <xacro:include filename="$(find mobile_base_description)/urdf/gazebo.xacro" />
+    <xacro:include filename="$(find mobile_base_description)/urdf/lidar.xacro" />
 </robot>
