Commit message: zx

File: src/mobile_base_description/urdf/mobile_base.urdf.xacro (robot description, xacro)
@@ -9,15 +9,15 @@
     <inertial>
       <origin
-        xyz="2.49993609215265E-05 -0.185259399389037 -0.00158375241138117"
-        rpy="0 0 0" />
-      <mass
-        value="7.12750649390085" />
-      <inertia
-        ixx="0.0457606455387283"
-        ixy="2.77322922063081E-06"
-        ixz="3.27411439344333E-05"
-        iyy="0.0218108431317148"
-        iyz="0.000878135124195838"
-        izz="0.0543254750685279" />
+        xyz="-0.00247544569007708 -0.188726144033008 -0.00331828982085067"
+        rpy="0 0 0" />
+      <mass
+        value="7.25669374827586" />
+      <inertia
+        ixx="0.0458578206362989"
+        ixy="2.77322922062842E-06"
+        ixz="3.27411439344336E-05"
+        iyy="0.0218763762344693"
+        iyz="0.000848533678871294"
+        izz="0.054377249546969" />
     </inertial>
     <visual>
@@ -49,15 +49,15 @@
     <inertial>
       <origin
-        xyz="0 0 0.035"
-        rpy="0 0 0" />
-      <mass
-        value="3.3906" />
-      <inertia
-        ixx="0.014535"
-        ixy="2.6574E-39"
-        ixz="-2.2718E-35"
-        iyy="0.014535"
-        iyz="-3.0837E-36"
-        izz="0.026345" />
+        xyz="0 0 1.38777878078145E-17"
+        rpy="0 0 0" />
+      <mass
+        value="4.46342151734513" />
+      <inertia
+        ixx="0.0214375253295535"
+        ixy="-9.27083006375532E-19"
+        ixz="-7.97975622392489E-20"
+        iyy="0.0214375253295535"
+        iyz="-1.43995601033231E-20"
+        izz="0.0375707416693319" />
     </inertial>
     <visual>
@@ -72,5 +72,5 @@
         name="">
         <color
-          rgba="0.79216 0.81961 0.93333 1" />
+          rgba="0.792156862745098 0.819607843137255 0.933333333333333 1" />
       </material>
     </visual>
@@ -89,5 +89,5 @@
     type="continuous">
     <origin
-      xyz="-0.167 0 0"
+      xyz="-0.137 0 0"
       rpy="1.5708 0 1.5708" />
     <parent
@@ -102,15 +102,15 @@
     <inertial>
       <origin
-        xyz="-1.3878E-17 -6.9389E-17 -0.035"
-        rpy="0 0 0" />
-      <mass
-        value="3.3906" />
-      <inertia
-        ixx="0.014535"
-        ixy="-2.8442E-19"
-        ixz="-3.179E-19"
-        iyy="0.014535"
-        iyz="-3.2069E-19"
-        izz="0.026345" />
+        xyz="-1.38777878078145E-17 -5.55111512312578E-17 2.77555756156289E-17"
+        rpy="0 0 0" />
+      <mass
+        value="4.46342151734513" />
+      <inertia
+        ixx="0.0214375253295535"
+        ixy="-2.9042607713123E-19"
+        ixz="-5.26009852170224E-19"
+        iyy="0.0214375253295535"
+        iyz="5.9105590148048E-20"
+        izz="0.0375707416693319" />
     </inertial>
     <visual>
@@ -125,5 +125,5 @@
         name="">
         <color
-          rgba="0.79216 0.81961 0.93333 1" />
+          rgba="0.792156862745098 0.819607843137255 0.933333333333333 1" />
       </material>
     </visual>
@@ -142,5 +142,5 @@
     type="continuous">
     <origin
-      xyz="0.167 0 0"
+      xyz="0.132 0 0"
       rpy="1.5708 0 1.5708" />
     <parent
@@ -155,15 +155,15 @@
     <inertial>
       <origin
-        xyz="-0.0063155 -0.0035273 -0.041077"
-        rpy="0 0 0" />
-      <mass
-        value="0.43416" />
-      <inertia
-        ixx="0.00031276"
-        ixy="-3.3539E-08"
-        ixz="-1.1302E-05"
-        iyy="0.00052583"
-        iyz="-1.4782E-05"
-        izz="0.00067509" />
+        xyz="-0.00631546895414616 -0.00352733963193702 -0.0410769894927615"
+        rpy="0 0 0" />
+      <mass
+        value="0.434157647657648" />
+      <inertia
+        ixx="0.000312761614867949"
+        ixy="-3.3538929303675E-08"
+        ixz="-1.13015683426856E-05"
+        iyy="0.000525827528394202"
+        iyz="-1.47821575025501E-05"
+        izz="0.000675087918007601" />
     </inertial>
     <visual>
@@ -178,5 +178,5 @@
         name="">
         <color
-          rgba="0.79216 0.81961 0.93333 1" />
+          rgba="0.792156862745098 0.819607843137255 0.933333333333333 1" />
       </material>
     </visual>
@@ -195,5 +195,5 @@
     type="fixed">
     <origin
-      xyz="0.00020041 0.27022 0.04328"
+      xyz="-0.0022996 0.27022 0.04328"
       rpy="2.3562 0 -3.1415" />
     <parent
@@ -208,15 +208,15 @@
     <inertial>
       <origin
-        xyz="-3.243E-05 0.03041 -0.00053785"
-        rpy="0 0 0" />
-      <mass
-        value="0.77573" />
-      <inertia
-        ixx="0.00093772"
-        ixy="3.8009E-07"
-        ixz="1.3264E-06"
-        iyy="0.00097173"
-        iyz="-1.5954E-06"
-        izz="0.00081322" />
+        xyz="-0.000537849970747462 3.24297391453357E-05 -0.0304099645492067"
+        rpy="0 0 0" />
+      <mass
+        value="0.77572976548165" />
+      <inertia
+        ixx="0.000813219708307499"
+        ixy="-1.32636836280717E-06"
+        ixz="1.59543719347388E-06"
+        iyy="0.000937718836199801"
+        iyz="3.80088779512422E-07"
+        izz="0.000971728129759389" />
     </inertial>
     <visual>
@@ -231,5 +231,5 @@
         name="">
         <color
-          rgba="0.79216 0.81961 0.93333 1" />
+          rgba="0.792156862745098 0.819607843137255 0.933333333333333 1" />
       </material>
     </visual>
@@ -248,6 +248,6 @@
     type="fixed">
     <origin
-      xyz="0 0.13302 -0.025212"
-      rpy="1.5708 0 3.1416" />
+      xyz="-0.0024966 0.13302 -0.025212"
+      rpy="-3.1416 0 1.5708" />
     <parent
       link="base_link" />

Commit message: sd

File: src/mobile_base_description/urdf/mobile_base.urdf.xacro (robot description, xacro)
@@ -9,5 +9,5 @@
     <inertial>
       <origin
-        xyz="-0.00247544569007708 -0.188726144033008 -0.00331828982085067"
+        xyz="-0.00247544569007708 -0.188726144033008 -0.00331828982085053"
         rpy="0 0 0" />
       <mass
@@ -15,8 +15,8 @@
       <inertia
         ixx="0.0458578206362989"
-        ixy="2.77322922062842E-06"
-        ixz="3.27411439344336E-05"
+        ixy="2.77322922062737E-06"
+        ixz="3.27411439344348E-05"
         iyy="0.0218763762344693"
-        iyz="0.000848533678871294"
+        iyz="0.000848533678871289"
         izz="0.054377249546969" />
     </inertial>
@@ -155,15 +155,15 @@
     <inertial>
       <origin
-        xyz="-0.00631546895414616 -0.00352733963193702 -0.0410769894927615"
-        rpy="0 0 0" />
-      <mass
-        value="0.434157647657648" />
-      <inertia
-        ixx="0.000312761614867949"
-        ixy="-3.3538929303675E-08"
-        ixz="-1.13015683426856E-05"
-        iyy="0.000525827528394202"
-        iyz="-1.47821575025501E-05"
-        izz="0.000675087918007601" />
+        xyz="-0.00744919022353967 -1.33048035397265E-06 -0.0345144672362048"
+        rpy="0 0 0" />
+      <mass
+        value="0.369842488759113" />
+      <inertia
+        ixx="0.000256169957334383"
+        ixy="-3.4750104335447E-08"
+        ixz="-1.13013119191708E-05"
+        iyy="0.00048809875532772"
+        iyz="-1.77820749757088E-08"
+        izz="0.000595013214946321" />
     </inertial>
     <visual>
@@ -195,6 +195,6 @@
     type="fixed">
     <origin
-      xyz="-0.0022996 0.27022 0.04328"
-      rpy="2.3562 0 -3.1415" />
+      xyz="-0.00229958657923851 0.270218938648069 0.043279647148146"
+      rpy="2.35619448960539 0 -3.14154419926722" />
     <parent
       link="base_link" />
@@ -208,5 +208,5 @@
     <inertial>
       <origin
-        xyz="-0.000537849970747462 3.24297391453357E-05 -0.0304099645492067"
+        xyz="-0.000537849970747406 3.24297391453357E-05 -0.0304099645492067"
         rpy="0 0 0" />
       <mass
@@ -214,8 +214,8 @@
       <inertia
         ixx="0.000813219708307499"
-        ixy="-1.32636836280717E-06"
-        ixz="1.59543719347388E-06"
+        ixy="-1.32636836280718E-06"
+        ixz="1.59543719347387E-06"
         iyy="0.000937718836199801"
-        iyz="3.80088779512422E-07"
+        iyz="3.80088779512424E-07"
         izz="0.000971728129759389" />
     </inertial>
@@ -257,3 +257,56 @@
       xyz="0 0 0" />
   </joint>
+  <link
+    name="crust_base_link">
+    <inertial>
+      <origin
+        xyz="-3.36265261816071E-08 0.0769069450394676 0.0161783208782746"
+        rpy="0 0 0" />
+      <mass
+        value="0.0643151587812771" />
+      <inertia
+        ixx="5.65916574952039E-05"
+        ixy="-7.18002494047286E-11"
+        ixz="-1.1856366830447E-11"
+        iyy="4.41373624530225E-05"
+        iyz="-2.11729650494233E-05"
+        izz="7.36661131733712E-05" />
+    </inertial>
+    <visual>
+      <origin
+        xyz="0 0 0"
+        rpy="0 0 0" />
+      <geometry>
+        <mesh
+          filename="file://$(find mobile_base_description)/meshes/crust_base_link.STL" />
+      </geometry>
+      <material
+        name="">
+        <color
+          rgba="0.792156862745098 0.819607843137255 0.933333333333333 1" />
+      </material>
+    </visual>
+    <collision>
+      <origin
+        xyz="0 0 0"
+        rpy="0 0 0" />
+      <geometry>
+        <mesh
+          filename="file://$(find mobile_base_description)/meshes/crust_base_link.STL" />
+      </geometry>
+    </collision>
+  </link>
+  <joint
+    name="crust_base_joint"
+    type="fixed">
+    <origin
+      xyz="-0.0025 0.12075 0.066"
+      rpy="0 0 0" />
+    <parent
+      link="base_link" />
+    <child
+      link="crust_base_link" />
+    <axis
+      xyz="0 0 0" />
+  </joint>
 </robot>
