Commit message: d

File: src/mobile_base_description/urdf/mobile_base_crust_old.urdf.xacro (robot description, xacro)
@@ -9,15 +9,15 @@
     <inertial>
       <origin
-        xyz="-0.188726144033008 0.00247544569007707 -0.00331828982085114"
-        rpy="0 0 0" />
-      <mass
-        value="7.25669374827584" />
-      <inertia
-        ixx="0.0218763762344693"
-        ixy="-2.77322922062719E-06"
-        ixz="0.000848533678871179"
-        iyy="0.0458578206362989"
-        iyz="-3.27411439344353E-05"
-        izz="0.0543772495469691" />
+        xyz="-0.00247544569007708 -0.188726144033008 -0.00331828982085053"
+        rpy="0 0 0" />
+      <mass
+        value="7.25669374827586" />
+      <inertia
+        ixx="0.0458578206362989"
+        ixy="2.77322922062737E-06"
+        ixz="3.27411439344348E-05"
+        iyy="0.0218763762344693"
+        iyz="0.000848533678871289"
+        izz="0.054377249546969" />
     </inertial>
     <visual>
@@ -49,15 +49,15 @@
     <inertial>
       <origin
-        xyz="0 0 -1.3878E-17"
-        rpy="0 0 0" />
-      <mass
-        value="4.4634" />
-      <inertia
-        ixx="0.021438"
-        ixy="9.2708E-19"
-        ixz="7.9798E-20"
-        iyy="0.021438"
-        iyz="-1.44E-20"
-        izz="0.037571" />
+        xyz="0 0 1.38777878078145E-17"
+        rpy="0 0 0" />
+      <mass
+        value="4.46342151734513" />
+      <inertia
+        ixx="0.0214375253295535"
+        ixy="-9.27083006375532E-19"
+        ixz="-7.97975622392489E-20"
+        iyy="0.0214375253295535"
+        iyz="-1.43995601033231E-20"
+        izz="0.0375707416693319" />
     </inertial>
     <visual>
@@ -72,5 +72,5 @@
         name="">
         <color
-          rgba="0.79216 0.81961 0.93333 1" />
+          rgba="0.792156862745098 0.819607843137255 0.933333333333333 1" />
       </material>
     </visual>
@@ -89,6 +89,6 @@
     type="continuous">
     <origin
-      xyz="0 0.137 0"
-      rpy="-1.5708 0 0" />
+      xyz="-0.137 0 0"
+      rpy="1.5708 0 1.5708" />
     <parent
       link="base_link" />
@@ -96,5 +96,5 @@
       link="left_wheel" />
     <axis
-      xyz="0 0 -1" />
+      xyz="0 0 1" />
   </joint>
   <link
@@ -102,15 +102,15 @@
     <inertial>
       <origin
-        xyz="-1.3878E-17 -5.5511E-17 2.7756E-17"
-        rpy="0 0 0" />
-      <mass
-        value="4.4634" />
-      <inertia
-        ixx="0.021438"
-        ixy="-2.9043E-19"
-        ixz="-5.2601E-19"
-        iyy="0.021438"
-        iyz="5.9106E-20"
-        izz="0.037571" />
+        xyz="-1.38777878078145E-17 -5.55111512312578E-17 2.77555756156289E-17"
+        rpy="0 0 0" />
+      <mass
+        value="4.46342151734513" />
+      <inertia
+        ixx="0.0214375253295535"
+        ixy="-2.9042607713123E-19"
+        ixz="-5.26009852170224E-19"
+        iyy="0.0214375253295535"
+        iyz="5.9105590148048E-20"
+        izz="0.0375707416693319" />
     </inertial>
     <visual>
@@ -125,5 +125,5 @@
         name="">
         <color
-          rgba="0.79216 0.81961 0.93333 1" />
+          rgba="0.792156862745098 0.819607843137255 0.933333333333333 1" />
       </material>
     </visual>
@@ -142,6 +142,6 @@
     type="continuous">
     <origin
-      xyz="0 -0.132 0"
-      rpy="1.5708 0 0" />
+      xyz="0.132 0 0"
+      rpy="1.5708 0 1.5708" />
     <parent
       link="base_link" />
@@ -155,15 +155,15 @@
     <inertial>
       <origin
-        xyz="-0.034514 -0.0074492 -1.0753E-06"
-        rpy="0 0 0" />
-      <mass
-        value="0.36984" />
-      <inertia
-        ixx="0.00059501"
-        ixy="-1.1301E-05"
-        ixz="-1.7395E-08"
-        iyy="0.00025617"
-        iyz="-2.6804E-08"
-        izz="0.0004881" />
+        xyz="-0.00744919022353967 -1.33048035397265E-06 -0.0345144672362048"
+        rpy="0 0 0" />
+      <mass
+        value="0.369842488759113" />
+      <inertia
+        ixx="0.000256169957334383"
+        ixy="-3.4750104335447E-08"
+        ixz="-1.13013119191708E-05"
+        iyy="0.00048809875532772"
+        iyz="-1.77820749757088E-08"
+        izz="0.000595013214946321" />
     </inertial>
     <visual>
@@ -178,5 +178,5 @@
         name="">
         <color
-          rgba="0.79216 0.81961 0.93333 1" />
+          rgba="0.792156862745098 0.819607843137255 0.933333333333333 1" />
       </material>
     </visual>
@@ -195,6 +195,6 @@
     type="fixed">
     <origin
-      xyz="0.27022 0.0022996 0.04328"
-      rpy="3.4262E-05 0.7854 4.8454E-05" />
+      xyz="-0.00229958657923851 0.270218938648069 0.043279647148146"
+      rpy="2.35619448960539 0 -3.14154419926722" />
     <parent
       link="base_link" />
@@ -205,18 +205,18 @@
   </joint>
   <link
-    name="laser">
-    <inertial>
-      <origin
-        xyz="-0.00053785 3.243E-05 -0.03041"
-        rpy="0 0 0" />
-      <mass
-        value="0.77573" />
-      <inertia
-        ixx="0.00081322"
-        ixy="-1.3264E-06"
-        ixz="1.5954E-06"
-        iyy="0.00093772"
-        iyz="3.8009E-07"
-        izz="0.00097173" />
+    name="scan">
+    <inertial>
+      <origin
+        xyz="-0.000537849970747406 3.24297391453357E-05 -0.0304099645492067"
+        rpy="0 0 0" />
+      <mass
+        value="0.77572976548165" />
+      <inertia
+        ixx="0.000813219708307499"
+        ixy="-1.32636836280718E-06"
+        ixz="1.59543719347387E-06"
+        iyy="0.000937718836199801"
+        iyz="3.80088779512424E-07"
+        izz="0.000971728129759389" />
     </inertial>
     <visual>
@@ -231,5 +231,5 @@
         name="">
         <color
-          rgba="0.79216 0.81961 0.93333 1" />
+          rgba="0.792156862745098 0.819607843137255 0.933333333333333 1" />
       </material>
     </visual>
@@ -245,31 +245,31 @@
   </link>
   <joint
-    name="laser_joint"
+    name="scan_joint"
     type="fixed">
     <origin
-      xyz="0.13302 0.0024966 -0.025212"
-      rpy="-3.1416 0 0" />
-    <parent
-      link="base_link" />
-    <child
-      link="laser" />
+      xyz="-0.0024966 0.13302 -0.025212"
+      rpy="-3.1416 0 1.5708" />
+    <parent
+      link="base_link" />
+    <child
+      link="scan" />
     <axis
       xyz="0 0 0" />
   </joint>
   <link
-    name="crust_base_link">
-    <inertial>
-      <origin
-        xyz="0 0 0"
-        rpy="0 0 0" />
-      <mass
-        value="0" />
-      <inertia
-        ixx="0"
-        ixy="0"
-        ixz="0"
-        iyy="0"
-        iyz="0"
-        izz="0" />
+    name="crust_base_link1">
+    <inertial>
+      <origin
+        xyz="-3.36265261816071E-08 0.0769069450394676 0.0161783208782746"
+        rpy="0 0 0" />
+      <mass
+        value="0.0643151587812771" />
+      <inertia
+        ixx="5.65916574952039E-05"
+        ixy="-7.18002494047286E-11"
+        ixz="-1.1856366830447E-11"
+        iyy="4.41373624530225E-05"
+        iyz="-2.11729650494233E-05"
+        izz="7.36661131733712E-05" />
     </inertial>
     <visual>
@@ -284,5 +284,5 @@
         name="">
         <color
-          rgba="1 1 1 1" />
+          rgba="0.792156862745098 0.819607843137255 0.933333333333333 1" />
       </material>
     </visual>
@@ -298,13 +298,13 @@
   </link>
   <joint
-    name="crust_base_joint"
+    name="crust_base_joint1"
     type="fixed">
     <origin
-      xyz="0.12075 0.0025 0.066"
-      rpy="0 0 -1.5708" />
-    <parent
-      link="base_link" />
-    <child
-      link="crust_base_link" />
+      xyz="-0.0025 0.12075 0.066"
+      rpy="0 0 0" />
+    <parent
+      link="base_link" />
+    <child
+      link="crust_base_link1" />
     <axis
       xyz="0 0 0" />
