Commit message: nu virker headless base real_base fake_base mm.

File: src/crust_arm_description/urdf/crust_arm_mobile.urdf.xacro (robot description, xacro)
@@ -5,17 +5,4 @@
 <robot
   name="crust_arm_mobile">
-  <joint
-    name="crust_base_joint"
-    type="fixed">
-    <origin
-      xyz="0 0 0"
-      rpy="0 0 0" />
-    <parent
-      link="crust_base_link1" />
-    <child
-      link="crust_base_link" />
-    <axis
-      xyz="0 0 0" />
-  </joint>
   <link
     name="crust_base_link">
@@ -40,5 +27,5 @@
       <geometry>
         <mesh
-          filename="file://$(find crust_arm_description)/meshes/base_link.STL" />
+          filename="file://$(find crust_arm_description)/meshes2/base_link.STL" />
       </geometry>
       <material

File: src/crust_arm_description/urdf/crust_arm_mobile_realsense.urdf.xacro (robot description, xacro)
@@ -4,7 +4,7 @@
      For more information, please see http://wiki.ros.org/sw_urdf_exporter -->
 <robot
-  name="Crust crawler version for urdf of crustcrawler new frame og reslsense">
-  <link
-    name="base_link">
+  name="crust_arm_mobile">
+  <link
+    name="crust_base_link">
     <inertial>
       <origin
@@ -27,19 +27,19 @@
       <geometry>
         <mesh
-          filename="package://Crust crawler version for urdf of crustcrawler new frame og reslsense/meshes/base_link.STL" />
-      </geometry>
-      <material
-        name="">
-        <color
-          rgba="0.89804 0.91765 0.92941 1" />
-      </material>
-    </visual>
-    <collision>
-      <origin
-        xyz="0 0 0"
-        rpy="0 0 0" />
-      <geometry>
-        <mesh
-          filename="package://Crust crawler version for urdf of crustcrawler new frame og reslsense/meshes/base_link.STL" />
+          filename="file://$(find crust_arm_description)/meshes/base_link.STL" />
+      </geometry>
+      <material
+        name="">
+        <color
+          rgba="0.89804 0.91765 0.92941 1" />
+      </material>
+    </visual>
+    <collision>
+      <origin
+        xyz="0 0 0"
+        rpy="0 0 0" />
+      <geometry>
+        <mesh
+          filename="file://$(find crust_arm_description)/meshes/base_link.STL" />
       </geometry>
     </collision>
@@ -67,19 +67,19 @@
       <geometry>
         <mesh
-          filename="package://Crust crawler version for urdf of crustcrawler new frame og reslsense/meshes/link_1.STL" />
-      </geometry>
-      <material
-        name="">
-        <color
-          rgba="0.89804 0.91765 0.92941 1" />
-      </material>
-    </visual>
-    <collision>
-      <origin
-        xyz="0 0 0"
-        rpy="0 0 0" />
-      <geometry>
-        <mesh
-          filename="package://Crust crawler version for urdf of crustcrawler new frame og reslsense/meshes/link_1.STL" />
+          filename="file://$(find crust_arm_description)/meshes/link_1.STL" />
+      </geometry>
+      <material
+        name="">
+        <color
+          rgba="0.89804 0.91765 0.92941 1" />
+      </material>
+    </visual>
+    <collision>
+      <origin
+        xyz="0 0 0"
+        rpy="0 0 0" />
+      <geometry>
+        <mesh
+          filename="file://$(find crust_arm_description)/meshes/link_1.STL" />
       </geometry>
     </collision>
@@ -92,5 +92,5 @@
       rpy="0 0 0" />
     <parent
-      link="base_link" />
+      link="crust_base_link" />
     <child
       link="link_1" />
@@ -125,19 +125,19 @@
       <geometry>
         <mesh
-          filename="package://Crust crawler version for urdf of crustcrawler new frame og reslsense/meshes/link_2.STL" />
-      </geometry>
-      <material
-        name="">
-        <color
-          rgba="0.89804 0.91765 0.92941 1" />
-      </material>
-    </visual>
-    <collision>
-      <origin
-        xyz="0 0 0"
-        rpy="0 0 0" />
-      <geometry>
-        <mesh
-          filename="package://Crust crawler version for urdf of crustcrawler new frame og reslsense/meshes/link_2.STL" />
+          filename="file://$(find crust_arm_description)/meshes/link_2.STL" />
+      </geometry>
+      <material
+        name="">
+        <color
+          rgba="0.89804 0.91765 0.92941 1" />
+      </material>
+    </visual>
+    <collision>
+      <origin
+        xyz="0 0 0"
+        rpy="0 0 0" />
+      <geometry>
+        <mesh
+          filename="file://$(find crust_arm_description)/meshes/link_2.STL" />
       </geometry>
     </collision>
@@ -183,19 +183,19 @@
       <geometry>
         <mesh
-          filename="package://Crust crawler version for urdf of crustcrawler new frame og reslsense/meshes/link_3.STL" />
-      </geometry>
-      <material
-        name="">
-        <color
-          rgba="0.89804 0.91765 0.92941 1" />
-      </material>
-    </visual>
-    <collision>
-      <origin
-        xyz="0 0 0"
-        rpy="0 0 0" />
-      <geometry>
-        <mesh
-          filename="package://Crust crawler version for urdf of crustcrawler new frame og reslsense/meshes/link_3.STL" />
+          filename="file://$(find crust_arm_description)/meshes/link_3.STL" />
+      </geometry>
+      <material
+        name="">
+        <color
+          rgba="0.89804 0.91765 0.92941 1" />
+      </material>
+    </visual>
+    <collision>
+      <origin
+        xyz="0 0 0"
+        rpy="0 0 0" />
+      <geometry>
+        <mesh
+          filename="file://$(find crust_arm_description)/meshes/link_3.STL" />
       </geometry>
     </collision>
@@ -241,19 +241,19 @@
       <geometry>
         <mesh
-          filename="package://Crust crawler version for urdf of crustcrawler new frame og reslsense/meshes/link_4.STL" />
-      </geometry>
-      <material
-        name="">
-        <color
-          rgba="0.89804 0.91765 0.92941 1" />
-      </material>
-    </visual>
-    <collision>
-      <origin
-        xyz="0 0 0"
-        rpy="0 0 0" />
-      <geometry>
-        <mesh
-          filename="package://Crust crawler version for urdf of crustcrawler new frame og reslsense/meshes/link_4.STL" />
+          filename="file://$(find crust_arm_description)/meshes/link_4.STL" />
+      </geometry>
+      <material
+        name="">
+        <color
+          rgba="0.89804 0.91765 0.92941 1" />
+      </material>
+    </visual>
+    <collision>
+      <origin
+        xyz="0 0 0"
+        rpy="0 0 0" />
+      <geometry>
+        <mesh
+          filename="file://$(find crust_arm_description)/meshes/link_4.STL" />
       </geometry>
     </collision>
@@ -299,5 +299,5 @@
       <geometry>
         <mesh
-          filename="package://Crust crawler version for urdf of crustcrawler new frame og reslsense/meshes/tool_link.STL" />
+          filename="file://$(find crust_arm_description)/meshes/tool_link.STL" />
       </geometry>
       <material
@@ -313,5 +313,5 @@
       <geometry>
         <mesh
-          filename="package://Crust crawler version for urdf of crustcrawler new frame og reslsense/meshes/tool_link.STL" />
+          filename="file://$(find crust_arm_description)/meshes/tool_link.STL" />
       </geometry>
     </collision>
@@ -330,5 +330,5 @@
       xyz="0 0 0" />
   </joint>
-  <link
+  <!--<link
     name="realsense_link">
     <inertial>
@@ -352,5 +352,5 @@
       <geometry>
         <mesh
-          filename="package://Crust crawler version for urdf of crustcrawler new frame og reslsense/meshes/realsense_link.STL" />
+          filename="file://$(find crust_arm_description)/meshes/realsense_link.STL" />
       </geometry>
       <material
@@ -366,5 +366,5 @@
       <geometry>
         <mesh
-          filename="package://Crust crawler version for urdf of crustcrawler new frame og reslsense/meshes/realsense_link.STL" />
+          filename="file://$(find crust_arm_description)/meshes/realsense_link.STL" />
       </geometry>
     </collision>
@@ -382,4 +382,4 @@
     <axis
       xyz="0 0 0" />
-  </joint>
+  </joint>-->
 </robot>

File: src/crust_arm_moveit_config/config/fake_base.xacro (robot description, xacro)
@@ -1,11 +1,11 @@
 <?xml version="1.0"?>
 <robot xmlns:xacro="http://www.ros.org/wiki/xacro" name="crust_arm_mobile">
-    <!--<xacro:arg name="initial_positions_file" default="initial_positions.yaml" />-->
+    <xacro:arg name="initial_positions_file" default="initial_positions.yaml" />
     <!-- Import panda urdf file -->
-    <!--<xacro:include filename="$(find crust_arm_description)/urdf/crust_arm_mobile.urdf.xacro" />-->
+    <xacro:include filename="$(find crust_arm_description)/urdf/crust_arm_mobile_realsense.urdf.xacro" />
     <!-- Import panda ros2_control description -->
-    <!--<xacro:include filename="crust.ros2_fake_control.xacro" />-->
-    <!--<xacro:crust_ros2_fake_control name="CrustFakeSystem" initial_positions_file="$(arg initial_positions_file)"/>-->
-        <!-- Import panda urdf file -->
+    <xacro:include filename="crust.ros2_fake_control.xacro" />
+    <xacro:crust_ros2_fake_control name="CrustFakeSystem" initial_positions_file="$(arg initial_positions_file)"/>
+    <xacro:include filename="crust_to_mobile_base.xacro" />
     <xacro:include filename="$(find mobile_base_description)/urdf/mobile_base_realsense.urdf.xacro" />
      <!-- Import panda urdf file -->

File: src/mobile_base_description/urdf/mobile_base_realsense.urdf.xacro (robot description, xacro)
@@ -4,5 +4,5 @@
      For more information, please see http://wiki.ros.org/sw_urdf_exporter -->
 <robot
-  name="mobile_base_assembly new real frames for crust with realsense">
+  name="crust_arm_mobile">
   <link
     name="base_link">
@@ -27,5 +27,5 @@
       <geometry>
         <mesh
-          filename="package://mobile_base_assembly new real frames for crust with realsense/meshes/base_link.STL" />
+          filename="file://$(find mobile_base_description)/meshes/base_link.STL" />
       </geometry>
       <material
@@ -41,5 +41,5 @@
       <geometry>
         <mesh
-          filename="package://mobile_base_assembly new real frames for crust with realsense/meshes/base_link.STL" />
+          filename="file://$(find mobile_base_description)/meshes/base_link.STL" />
       </geometry>
     </collision>
@@ -67,19 +67,19 @@
       <geometry>
         <mesh
-          filename="package://mobile_base_assembly new real frames for crust with realsense/meshes/left_wheel.STL" />
-      </geometry>
-      <material
-        name="">
-        <color
-          rgba="0.79216 0.81961 0.93333 1" />
-      </material>
-    </visual>
-    <collision>
-      <origin
-        xyz="0 0 0"
-        rpy="0 0 0" />
-      <geometry>
-        <mesh
-          filename="package://mobile_base_assembly new real frames for crust with realsense/meshes/left_wheel.STL" />
+          filename="file://$(find mobile_base_description)/meshes/left_wheel.STL" />
+      </geometry>
+      <material
+        name="">
+        <color
+          rgba="0.79216 0.81961 0.93333 1" />
+      </material>
+    </visual>
+    <collision>
+      <origin
+        xyz="0 0 0"
+        rpy="0 0 0" />
+      <geometry>
+        <mesh
+          filename="file://$(find mobile_base_description)/meshes/left_wheel.STL" />
       </geometry>
     </collision>
@@ -120,19 +120,19 @@
       <geometry>
         <mesh
-          filename="package://mobile_base_assembly new real frames for crust with realsense/meshes/right_wheel.STL" />
-      </geometry>
-      <material
-        name="">
-        <color
-          rgba="0.79216 0.81961 0.93333 1" />
-      </material>
-    </visual>
-    <collision>
-      <origin
-        xyz="0 0 0"
-        rpy="0 0 0" />
-      <geometry>
-        <mesh
-          filename="package://mobile_base_assembly new real frames for crust with realsense/meshes/right_wheel.STL" />
+          filename="file://$(find mobile_base_description)/meshes/right_wheel.STL" />
+      </geometry>
+      <material
+        name="">
+        <color
+          rgba="0.79216 0.81961 0.93333 1" />
+      </material>
+    </visual>
+    <collision>
+      <origin
+        xyz="0 0 0"
+        rpy="0 0 0" />
+      <geometry>
+        <mesh
+          filename="file://$(find mobile_base_description)/meshes/right_wheel.STL" />
       </geometry>
     </collision>
@@ -173,19 +173,19 @@
       <geometry>
         <mesh
-          filename="package://mobile_base_assembly new real frames for crust with realsense/meshes/camera.STL" />
-      </geometry>
-      <material
-        name="">
-        <color
-          rgba="0.79216 0.81961 0.93333 1" />
-      </material>
-    </visual>
-    <collision>
-      <origin
-        xyz="0 0 0"
-        rpy="0 0 0" />
-      <geometry>
-        <mesh
-          filename="package://mobile_base_assembly new real frames for crust with realsense/meshes/camera.STL" />
+          filename="file://$(find mobile_base_description)/meshes/camera.STL" />
+      </geometry>
+      <material
+        name="">
+        <color
+          rgba="0.79216 0.81961 0.93333 1" />
+      </material>
+    </visual>
+    <collision>
+      <origin
+        xyz="0 0 0"
+        rpy="0 0 0" />
+      <geometry>
+        <mesh
+          filename="file://$(find mobile_base_description)/meshes/camera.STL" />
       </geometry>
     </collision>
@@ -226,19 +226,19 @@
       <geometry>
         <mesh
-          filename="package://mobile_base_assembly new real frames for crust with realsense/meshes/scan.STL" />
-      </geometry>
-      <material
-        name="">
-        <color
-          rgba="0.79216 0.81961 0.93333 1" />
-      </material>
-    </visual>
-    <collision>
-      <origin
-        xyz="0 0 0"
-        rpy="0 0 0" />
-      <geometry>
-        <mesh
-          filename="package://mobile_base_assembly new real frames for crust with realsense/meshes/scan.STL" />
+          filename="file://$(find mobile_base_description)/meshes/scan.STL" />
+      </geometry>
+      <material
+        name="">
+        <color
+          rgba="0.79216 0.81961 0.93333 1" />
+      </material>
+    </visual>
+    <collision>
+      <origin
+        xyz="0 0 0"
+        rpy="0 0 0" />
+      <geometry>
+        <mesh
+          filename="file://$(find mobile_base_description)/meshes/scan.STL" />
       </geometry>
     </collision>
@@ -279,19 +279,19 @@
       <geometry>
         <mesh
-          filename="package://mobile_base_assembly new real frames for crust with realsense/meshes/crust_base_link1.STL" />
-      </geometry>
-      <material
-        name="">
-        <color
-          rgba="0.79216 0.81961 0.93333 1" />
-      </material>
-    </visual>
-    <collision>
-      <origin
-        xyz="0 0 0"
-        rpy="0 0 0" />
-      <geometry>
-        <mesh
-          filename="package://mobile_base_assembly new real frames for crust with realsense/meshes/crust_base_link1.STL" />
+          filename="file://$(find mobile_base_description)/meshes/crust_base_link.STL" />
+      </geometry>
+      <material
+        name="">
+        <color
+          rgba="0.79216 0.81961 0.93333 1" />
+      </material>
+    </visual>
+    <collision>
+      <origin
+        xyz="0 0 0"
+        rpy="0 0 0" />
+      <geometry>
+        <mesh
+          filename="file://$(find mobile_base_description)/meshes/crust_base_link.STL" />
       </geometry>
     </collision>
