Commit message: æ lort virker

File: src/crust_arm_description/urdf/crust_arm_mobile_w_gripper.urdf.xacro (robot description, xacro)
@@ -107,15 +107,15 @@
     <inertial>
       <origin
-        xyz="0.00088105 -0.16138 -0.00028433"
-        rpy="0 0 0" />
-      <mass
-        value="0.11516" />
-      <inertia
-        ixx="8.1961E-05"
-        ixy="-1.5264E-08"
-        ixz="4.1398E-13"
-        iyy="2.8324E-05"
-        iyz="-8.8059E-07"
-        izz="7.0335E-05" />
+        xyz="-0.000963145876619109 -0.161378299147481 -0.000284331859152033"
+        rpy="0 0 0" />
+      <mass
+        value="0.115162829413528" />
+      <inertia
+        ixx="8.19607421534774E-05"
+        ixy="-1.52641760422517E-08"
+        ixz="4.13979918627638E-13"
+        iyy="2.83238373910903E-05"
+        iyz="-8.80590794460533E-07"
+        izz="7.03346423289087E-05" />
     </inertial>
     <visual>
@@ -130,5 +130,5 @@
         name="">
         <color
-          rgba="0.89804 0.91765 0.92941 1" />
+          rgba="0.898039215686275 0.917647058823529 0.929411764705882 1" />
       </material>
     </visual>
@@ -143,9 +143,9 @@
     </collision>
   </link>
-  <!--<joint
+  <joint
     name="joint_2"
     type="revolute">
     <origin
-      xyz="-0.0018442 -0.00315 0.0576"
+      xyz="0 -0.00315 0.0576"
       rpy="-1.5708 0 0" />
     <parent
@@ -154,23 +154,5 @@
       link="link_2" />
     <axis
-      xyz="-0.075311 0 0.99716" />
-    <limit
-      lower="-2.2"
-      upper="2.2"
-      effort="200"
-      velocity="3" />
-  </joint>-->
-  <joint
-    name="joint_2"
-    type="revolute">
-    <origin
-      xyz="-0.00184419164302273 -0.00314999999999882 0.0575999999999965"
-      rpy="-1.5707963267949 0 0" />
-    <parent
-      link="link_1" />
-    <child
-      link="link_2" />
-    <axis
-      xyz="-0.0753114848976472 0 0.99716005748451" />
+      xyz="0 0 1" />
     <limit
       lower="-2.2"
@@ -219,9 +201,9 @@
     </collision>
   </link>
-  <!--<joint
+  <joint
     name="joint_3"
     type="revolute">
     <origin
-      xyz="0.0018442 -0.2198 -0.003"
+      xyz="0 -0.2198 -0.003"
       rpy="0 0 0" />
     <parent
@@ -236,15 +218,55 @@
       effort="200"
       velocity="3" />
-  </joint>-->
-  <joint
-    name="joint_3"
+  </joint>
+  <link
+    name="link_4">
+    <inertial>
+      <origin
+        xyz="-5.2458E-15 -0.017324 -4.8711E-15"
+        rpy="0 0 0" />
+      <mass
+        value="0.012733" />
+      <inertia
+        ixx="5.3648E-06"
+        ixy="-6.1775E-22"
+        ixz="3.5043E-21"
+        iyy="4.553E-06"
+        iyz="9.8621E-21"
+        izz="2.0871E-06" />
+    </inertial>
+    <visual>
+      <origin
+        xyz="0 0 0"
+        rpy="0 0 0" />
+      <geometry>
+        <mesh
+          filename="file://$(find crust_arm_description)/meshes_gripper/link_4.STL" />
+      </geometry>
+      <material
+        name="">
+        <color
+          rgba="0.89804 0.91765 0.92941 1" />
+      </material>
+    </visual>
+    <collision>
+      <origin
+        xyz="0 0 0"
+        rpy="0 0 0" />
+      <geometry>
+        <mesh
+          filename="file://$(find crust_arm_description)/meshes_gripper/link_4.STL" />
+      </geometry>
+    </collision>
+  </link>
+  <joint
+    name="joint_4"
     type="revolute">
     <origin
-      xyz="0.00184419164302234 -0.2198 -0.00299999999999676"
+      xyz="0 -0.2208 -0.003"
       rpy="0 0 0" />
     <parent
-      link="link_2" />
-    <child
       link="link_3" />
+    <child
+      link="link_4" />
     <axis
       xyz="0 0 1" />
@@ -256,53 +278,228 @@
   </joint>
   <link
-    name="link_4">
-    <inertial>
-      <origin
-        xyz="-1.0547E-14 -0.017324 -9.1593E-16"
-        rpy="0 0 0" />
-      <mass
-        value="0.012733" />
-      <inertia
-        ixx="5.3648E-06"
-        ixy="-6.7106E-22"
-        ixz="-3.9867E-22"
-        iyy="4.553E-06"
-        iyz="1.1243E-20"
-        izz="2.0871E-06" />
-    </inertial>
-    <visual>
-      <origin
-        xyz="0 0 0"
-        rpy="0 0 0" />
-      <geometry>
-        <mesh
-          filename="file://$(find crust_arm_description)/meshes_gripper/link_4.STL" />
-      </geometry>
-      <material
-        name="">
-        <color
-          rgba="0.89804 0.91765 0.92941 1" />
-      </material>
-    </visual>
-    <collision>
-      <origin
-        xyz="0 0 0"
-        rpy="0 0 0" />
-      <geometry>
-        <mesh
-          filename="file://$(find crust_arm_description)/meshes_gripper/link_4.STL" />
-      </geometry>
-    </collision>
-  </link>
-  <joint
-    name="joint_4"
+    name="flange_link">
+    <inertial>
+      <origin
+        xyz="0.0017146 -6.5642E-15 -3.0531E-16"
+        rpy="0 0 0" />
+      <mass
+        value="0.0029645" />
+      <inertia
+        ixx="5.4073E-07"
+        ixy="1.0659E-22"
+        ixz="1.8551E-22"
+        iyy="4.0167E-07"
+        iyz="5.1627E-22"
+        izz="1.6602E-07" />
+    </inertial>
+    <visual>
+      <origin
+        xyz="0 0 0"
+        rpy="0 0 0" />
+      <geometry>
+        <mesh
+          filename="file://$(find crust_arm_description)/meshes_gripper/flange_link.STL" />
+      </geometry>
+      <material
+        name="">
+        <color
+          rgba="0.89804 0.91765 0.92941 1" />
+      </material>
+    </visual>
+    <collision>
+      <origin
+        xyz="0 0 0"
+        rpy="0 0 0" />
+      <geometry>
+        <mesh
+          filename="file://$(find crust_arm_description)/meshes_gripper/flange_link.STL" />
+      </geometry>
+    </collision>
+  </link>
+  <joint
+    name="flange_joint"
+    type="fixed">
+    <origin
+      xyz="0 -0.0385 0"
+      rpy="1.5708 0 -1.5708" />
+    <parent
+      link="link_4" />
+    <child
+      link="flange_link" />
+    <axis
+      xyz="0 0 0" />
+  </joint>
+  <link
+    name="camera_link">
+    <inertial>
+      <origin
+        xyz="-0.0094472 -0.017953 -0.0015914"
+        rpy="0 0 0" />
+      <mass
+        value="0.12525" />
+      <inertia
+        ixx="8.5958E-05"
+        ixy="-1.7858E-08"
+        ixz="-5.2292E-07"
+        iyy="1.3969E-05"
+        iyz="2.3752E-10"
+        izz="7.897E-05" />
+    </inertial>
+    <visual>
+      <origin
+        xyz="0 0 0"
+        rpy="0 0 0" />
+      <geometry>
+        <mesh
+          filename="file://$(find crust_arm_description)/meshes_gripper/camera_link.STL" />
+      </geometry>
+      <material
+        name="">
+        <color
+          rgba="0.79216 0.81961 0.93333 1" />
+      </material>
+    </visual>
+    <collision>
+      <origin
+        xyz="0 0 0"
+        rpy="0 0 0" />
+      <geometry>
+        <mesh
+          filename="file://$(find crust_arm_description)/meshes_gripper/camera_link.STL" />
+      </geometry>
+    </collision>
+  </link>
+  <joint
+    name="camera_joint"
+    type="fixed">
+    <origin
+      xyz="0.0288 0.017962 0.055"
+      rpy="0 0 0" />
+    <parent
+      link="flange_link" />
+    <child
+      link="camera_link" />
+    <axis
+      xyz="0 0 0" />
+  </joint>
+  <link
+    name="tool_link">
+    </link>
+  <joint
+    name="tool_joint"
+    type="fixed">
+    <origin
+      xyz="0.12831 0 0"
+      rpy="0 0 0" />
+    <parent
+      link="flange_link" />
+    <child
+      link="tool_link" />
+    <axis
+      xyz="0 0 0" />
+  </joint>
+  <link
+    name="gripper_link">
+    <inertial>
+      <origin
+        xyz="0.029256 4.8004E-09 -3.0878E-05"
+        rpy="0 0 0" />
+      <mass
+        value="0.089066" />
+      <inertia
+        ixx="1.5005E-05"
+        ixy="-5.9945E-13"
+        ixz="-3.6548E-07"
+        iyy="2.4693E-05"
+        iyz="-1.0592E-11"
+        izz="2.1002E-05" />
+    </inertial>
+    <visual>
+      <origin
+        xyz="0 0 0"
+        rpy="0 0 0" />
+      <geometry>
+        <mesh
+          filename="file://$(find crust_arm_description)/meshes_gripper/gripper_link.STL" />
+      </geometry>
+      <material
+        name="">
+        <color
+          rgba="0.20784 0.20784 0.20784 1" />
+      </material>
+    </visual>
+    <collision>
+      <origin
+        xyz="0 0 0"
+        rpy="0 0 0" />
+      <geometry>
+        <mesh
+          filename="file://$(find crust_arm_description)/meshes_gripper/gripper_link.STL" />
+      </geometry>
+    </collision>
+  </link>
+  <joint
+    name="gripper_joint"
+    type="fixed">
+    <origin
+      xyz="0 0 0"
+      rpy="0 0 0" />
+    <parent
+      link="flange_link" />
+    <child
+      link="gripper_link" />
+    <axis
+      xyz="0 0 0" />
+  </joint>
+  <link
+    name="finger1_link">
+    <inertial>
+      <origin
+        xyz="0.00064145 -0.040478 -3.636E-15"
+        rpy="0 0 0" />
+      <mass
+        value="0.024008" />
+      <inertia
+        ixx="8.2624E-06"
+        ixy="1.6564E-07"
+        ixz="-1.6873E-23"
+        iyy="4.9212E-06"
+        iyz="-2.1007E-20"
+        izz="4.8948E-06" />
+    </inertial>
+    <visual>
+      <origin
+        xyz="0 0 0"
+        rpy="0 0 0" />
+      <geometry>
+        <mesh
+          filename="file://$(find crust_arm_description)/meshes_gripper/finger1_link.STL" />
+      </geometry>
+      <material
+        name="">
+        <color
+          rgba="0.89804 0.91765 0.92941 1" />
+      </material>
+    </visual>
+    <collision>
+      <origin
+        xyz="0 0 0"
+        rpy="0 0 0" />
+      <geometry>
+        <mesh
+          filename="file://$(find crust_arm_description)/meshes_gripper/finger1_link.STL" />
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
Commit message: æ lort virker i virkeligheden også

File: src/crust_arm_description/urdf/crust_arm_mobile_w_gripper.urdf.xacro (robot description, xacro)
@@ -561,5 +561,5 @@
       link="finger2_link" />
     <axis
-      xyz="0 0 -1" />
+      xyz="0 0 1" />
     <limit
       lower="-2.2"
@@ -567,8 +567,8 @@
       effort="200"
       velocity="3" />
-    <mimic
+    <!--<mimic
       joint="finger1_joint"
-      multiplier="1"
-      offset="0" />
+      multiplier="-1"
+      offset="0" />-->
   </joint>
 </robot>

File: src/crust_arm_moveit_config/config/crust_gripper.ros2_control.xacro (robot description, xacro)
@@ -43,5 +43,5 @@
       </joint>
       <joint name="finger1_joint">
-        <param name="id">4</param>
+        <param name="id">6</param>
         <command_interface name="position"/>
         <command_interface name="velocity"/>
@@ -51,7 +51,7 @@
       </joint>
       <joint name="finger2_joint">
-        <param name="id">6</param>
-        <param name="mimic">finger1_joint</param>
-        <param name="multiplier">-1</param>
+        <param name="id">4</param>
+        <!--<param name="mimic">finger1_joint</param>-->
+        <!--<param name="multiplier">-1</param>-->
         <command_interface name="position"/>
         <command_interface name="velocity"/>

Commit message: asf

File: src/crust_arm_description/urdf/crust_arm_mobile_w_gripper.urdf.xacro (robot description, xacro)
@@ -380,4 +380,20 @@
     <child
       link="camera_link" />
+    <axis
+      xyz="0 0 0" />
+  </joint>
+  <link
+    name="workspace_center">
+    </link>
+  <joint
+    name="workspace_center_joint"
+    type="fixed">
+    <origin
+      xyz="0.32 0 0"
+      rpy="0 0 0" />
+    <parent
+      link="crust_base_link" />
+    <child
+      link="workspace_center" />
     <axis
       xyz="0 0 0" />

File: src/mobile_base_description/urdf/mobile_base_realsense.urdf.xacro (robot description, xacro)
@@ -192,5 +192,5 @@
   </link>
   <joint
-    name="camera_joint"
+    name="camera_joint1"
     type="fixed">
     <origin
